File: BirtdayCard.kicad_pcb.kicad_pcb (KiCad board)
At the start: 2 copper layers, 150 x 150 mm, 59 parts, among them J2 Conn_01x05_Pin, J3 USB_C_Receptacle_USB2.0, Q1 2N7002_C306856, U1 ESP32-C3-WROOM-02-N4(4MB), U2 AMS1117-3.3_C347222

Commit message: Concept 1 PCB
Parts:
- added G***: LOGO, LOGO, F.Cu at (132.0, 151.0)
- REF**: moved to F.Cu
- moved C14 117.2 mm to (252.4, 122.4)
- moved C15 117.2 mm to (213.3, 119.9)
- moved C16 117.2 mm to (194.1, 94.9)
- moved C17 117.2 mm to (213.3, 122.9)
- moved C32 117.2 mm to (218.1, 125.9)
- moved D10 117.2 mm to (273.8, 85.0)
- moved D11 117.2 mm to (273.8, 91.4)
- moved D12 117.2 mm to (273.8, 97.8)
- moved D13 117.2 mm to (273.8, 104.3)
- moved D14 117.2 mm to (273.8, 110.8)
- moved D20 117.2 mm to (238.3, 133.1)
- moved D21 117.2 mm to (238.3, 140.1)
- moved D22 117.2 mm to (238.3, 147.2)
- moved D23 117.2 mm to (238.3, 154.2)
- moved D24 117.2 mm to (238.3, 161.2)
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Other:
- board text added: "Lieve Sander, Wauw, 18 jaar oud! Nu ben je officieel volwassen, wat betekent dat je allemaal nieuwe features hebt unlocked in de gezamenlijke server. Even op een rijtje: 1. Full access to the worldmap 2. Een eigen stem (waar misschien naar wordt geluisterd!) 3. Je eigen zorgverZEKERING én andere vaste lasten! 4. Toegang tot de vierwielige fatbike crusher (wanneer je dat plastic kaartje hebt gesco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"
- board text removed: "Lieve Sander, Wauw, 18 jaar oud! Nu ben je officieel volwassen, wat betekent dat je allemaal nieuwe features hebt unlocked in de gezamenlijke server. Even op een rijtje: 1. Full access to the worldmap 2. Een eigen stem (waar misschien naar wordt geluisterd!) 3. Je eigen zorgverZEKERING én andere vaste lasten! 4. Toegang tot de vierwielige fatbike crusher (wanneer je een plastic kaartje hebt gesco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"
