File: bom/BirtdayCard.kicad_pcb.kicad_pcb (KiCad board)
At the start: 2 copper layers, 150 x 150 mm, 56 parts, among them J1 Conn_01x04_Socket, J2 Conn_01x05_Pin, Q1 2N7002_C306856, U1 ESP32-C3-WROOM-02-N4(4MB), U2 AMS1117-3.3_C347222

Commit message: board improvements and added media
Parts:
- moved D5 0.50 mm to (143.5, 113.0)
- moved G*** 0.50 mm to (131.0, 124.0), turned to -45 degrees
Other:
- board text added: "Lieve Sander,"
- board text removed: ","
- board text removed: "Lieve"
- board text removed: "Sander"
